File: Blackbox v2.0/hardware/untitled.brd (EAGLE design)
At the start: 63.9 x 41.6 mm, 40 parts, among them IC1 MEGA8-AI, IC2 7805DT, Q1 CSM-7X-DU

Commit message: Adaug placa in versiunea noua
(mufa de programare cu 6 pini si condensator pt ADC)
Parts:
- added C3: 22p, resistor:C0805
- JP1: device SparkFun-Connectors:1X05 -> SparkFun-Connectors:1X06
Connections:
- removed net AVCC: IC1.18
- new net N$38: C3.2, IC1.20
- net +5V: now also IC1.18, JP1.6
- net GND: now also C3.1
Routing:
- net +5V: track 185.7 -> 205.5 mm, vias 9 -> 10
- net GND: track 136.7 -> 139.2 mm
- net N$38: track 0.00 -> 2.11 mm
Changed lines of the file:
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@@
 <element name="R2" library="resistor" package="R0805" value="" x="46" y="2.8"/>
 <element name="R3" library="resistor" package="R0805" value="" x="42" y="2.8"/>
-<element name="JP1" library="SparkFun-Connectors" package="1X05" value="" x="30.8" y="7.2" rot="R90"/>
 <element name="U$2" library="drv8833" package="PW" value="DRV8833-PWP" x="38.8" y="29.2"/>
 <element name="R4" library="resistor" package="R0805" value="33k" x="44" y="32"/>
@@
 <element name="C7" library="resistor" package="C0805" value="10nF" x="54.4" y="21.19"/>
 <element name="C8" library="resistor" package="C0805" value="2.2uF" x="58.28" y="21.19" rot="R180"/>
+<element name="C3" library="resistor" package="C0805" value="22p" x="26.8" y="17.2" rot="R270"/>
+<element name="JP1" library="SparkFun-Connectors" package="1X06" value="" x="30.8" y="7.2" rot="R90"/>
 </elements>
 <signals>
-<signal name="AVCC">
-<contactref element="IC1" pad="18"/>
-</signal>
 <signal name="GND">
 <contactref element="IC1" pad="3"/>
@@
 <contactref element="U$1" pad="GND"/>
 <contactref element="R3" pad="1"/>
-<contactref element="JP1" pad="5"/>
 <wire x1="24.6926" y1="17.2" x2="20" y2="17.2" width="0.4064" layer="1"/>
 <wire x1="20" y1="17.2" x2="19.6" y2="16.8" width="0.4064" layer="1"/>
@@
 <wire x1="37.825" y1="35.775" x2="36.4" y2="37.2" width="0.4064" layer="1"/>
 <wire x1="36.4" y1="37.2" x2="34" y2="39.6" width="1.27" layer="1"/>
+<contactref element="C3" pad="1"/>
+<wire x1="26.8" y1="18.05" x2="26.45" y2="18.05" width="0.4064" layer="1"/>
+<wire x1="26.45" y1="18.05" x2="25.6" y2="17.2" width="0.4064" layer="1"/>
+<wire x1="25.6" y1="17.2" x2="24.6926" y2="17.2" width="0.4064" layer="1"/>
+<contactref element="JP1" pad="5"/>
 <wire x1="16" y1="18" x2="16.1074" y2="18" width="0" layer="19" extent="1-1"/>
 </signal>
@@
 <wire x1="48.4" y1="31.6" x2="48.4" y2="28.05" width="0.4064" layer="1"/>
 <wire x1="48.4" y1="28.05" x2="48.35" y2="28" width="0.4064" layer="1"/>
+<contactref element="IC1" pad="18"/>
+<wire x1="16.1074" y1="15.6" x2="21.6" y2="15.6" width="0.4064" layer="1"/>
+<wire x1="21.6" y1="15.6" x2="22.4" y2="14.8" width="0.4064" layer="1"/>
+<wire x1="22.4" y1="14.8" x2="24.6926" y2="14.8" width="0.4064" layer="1"/>
+<contactref element="JP1" pad="6"/>
+<wire x1="28" y1="14.8" x2="24.6926" y2="14.8" width="0.4064" layer="1"/>
+<wire x1="28" y1="14.8" x2="28.4" y2="15.2" width="0.4064" layer="1"/>
+<wire x1="28.4" y1="15.2" x2="28.4" y2="19.6" width="0.4064" layer="1"/>
+<wire x1="28.4" y1="19.6" x2="28.8" y2="20" width="0.4064" layer="1"/>
+<via x="28.8" y="20" extent="1-16" drill="0.6" shape="square"/>
+<wire x1="28.8" y1="20" x2="30.7" y2="20" width="1.27" layer="16"/>
+<wire x1="30.7" y1="20" x2="30.8" y2="19.9" width="0.4064" layer="16"/>
 </signal>
 <signal name="RESET">
 <contactref element="IC1" pad="29"/>
 <contactref element="R1" pad="1"/>
-<contactref element="JP1" pad="4"/>
 <via x="20" y="24" extent="1-16" drill="0.6" diameter="1" shape="square"/>
 <wire x1="27.58" y1="14.82" x2="25.6" y2="16.4" width="1.27" layer="16"/>
@@
 <wire x1="25.6" y1="20.8" x2="22.4" y2="24" width="1.27" layer="16"/>
 <wire x1="22.4" y1="24" x2="20" y2="24" width="1.27" layer="16"/>
-<wire x1="30.8" y1="14.82" x2="27.58" y2="14.82" width="1.27" layer="16"/>
 <wire x1="20" y1="21.0926" x2="20" y2="24" width="0.4064" layer="1"/>
 <wire x1="19.2" y1="25.55" x2="19.2" y2="24.8" width="0.4064" layer="1"/>
 <wire x1="19.2" y1="24.8" x2="20" y2="24" width="0.4064" layer="1"/>
+<contactref element="JP1" pad="4"/>
+<wire x1="30.8" y1="14.82" x2="27.58" y2="14.82" width="1.27" layer="16"/>
 </signal>
 <signal name="N$1">
@@
 <wire x1="17.2" y1="36.94" x2="21.6" y2="36.94" width="1.27" layer="1"/>
 <via x="24" y="26" extent="1-16" drill="0.6" diameter="1" shape="square"/>
-<wire x1="24" y1="26" x2="29.6" y2="20" width="1.27" layer="16"/>
-<wire x1="29.6" y1="20" x2="33.2" y2="20" width="1.27" layer="16"/>
-<wire x1="33.2" y1="20" x2="44.8" y2="8.4" width="1.27" layer="16"/>
-<wire x1="44.8" y1="8.4" x2="46.8" y2="8.4" width="1.27" layer="16"/>
+<wire x1="24" y1="26" x2="27.6" y2="22.4" width="1.27" layer="16"/>
+<wire x1="27.6" y1="22.4" x2="31.6" y2="22.4" width="1.27" layer="16"/>
+<wire x1="31.6" y1="22.4" x2="45.2" y2="8.4" width="1.27" layer="16"/>
+<wire x1="45.2" y1="8.4" x2="46.8" y2="8.4" width="1.27" layer="16"/>
 <wire x1="21.6" y1="36.94" x2="21.6" y2="36.4" width="0.4064" layer="1"/>
 <wire x1="21.6" y1="36.4" x2="25.6" y2="32.4" width="0.4064" layer="1"/>
@@
 <signal name="N$4">
 <contactref element="IC1" pad="17"/>
-<contactref element="JP1" pad="3"/>
 <via x="27.2" y="12.4" extent="1-16" drill="1" diameter="1.5" shape="square"/>
 <wire x1="24.6926" y1="14" x2="25.6" y2="14" width="0.4064" layer="1"/>
 <wire x1="25.6" y1="14" x2="27.2" y2="12.4" width="0.4064" layer="1"/>
+<contactref element="JP1" pad="3"/>
 <wire x1="30.8" y1="12.28" x2="27.32" y2="12.28" width="1.27" layer="16"/>
 <wire x1="27.32" y1="12.28" x2="27.2" y2="12.4" width="1.27" layer="16"/>
@@
 <signal name="N$5">
 <contactref element="IC1" pad="16"/>
-<contactref element="JP1" pad="2"/>
 <via x="27.2" y="9.6" extent="1-16" drill="1" diameter="1.5" shape="square"/>
 <wire x1="23.2" y1="12.5074" x2="23.2" y2="10.4" width="0.4064" layer="1"/>
 <wire x1="23.2" y1="10.4" x2="24" y2="9.6" width="0.4064" layer="1"/>
 <wire x1="24" y1="9.6" x2="27.2" y2="9.6" width="0.4064" layer="1"/>
+<contactref element="JP1" pad="2"/>
 <wire x1="30.8" y1="9.74" x2="27.34" y2="9.74" width="1.27" layer="16"/>
 <wire x1="27.34" y1="9.74" x2="27.2" y2="9.6" width="1.27" layer="16"/>
@@
 <signal name="N$6">
 <contactref element="IC1" pad="15"/>
-<contactref element="JP1" pad="1"/>
 <via x="27.2" y="7.2" extent="1-16" drill="1" diameter="1.5" shape="square"/>
 <wire x1="22.4" y1="12.5074" x2="22.4" y2="8.4" width="0.4064" layer="1"/>
 <wire x1="22.4" y1="8.4" x2="23.6" y2="7.2" width="0.4064" layer="1"/>
 <wire x1="23.6" y1="7.2" x2="27.2" y2="7.2" width="0.4064" layer="1"/>
+<contactref element="JP1" pad="1"/>
 <wire x1="27.2" y1="7.2" x2="30.8" y2="7.2" width="1.27" layer="16"/>
 </signal>
@@
 <contactref element="U$2" pad="9"/>
 <contactref element="IC1" pad="24"/>
-<wire x1="24.6926" y1="19.6" x2="29.6" y2="19.6" width="0.4064" layer="1"/>
 <via x="33.6" y="23.6" extent="1-16" drill="1" shape="square"/>
 <wire x1="33.6" y1="23.6" x2="44" y2="23.6" width="1.27" layer="16"/>
@@
 <wire x1="44" y1="24.8" x2="42.4" y2="26.4" width="0.4064" layer="1"/>
 <wire x1="41.075" y1="26.4" x2="42.4" y2="26.4" width="0.4064" layer="1"/>
-<wire x1="29.6" y1="19.6" x2="33.6" y2="23.6" width="0.4064" layer="1"/>
 <wire x1="36.525" y1="26.4" x2="36.4" y2="26.4" width="0.4064" layer="1"/>
 <wire x1="36.4" y1="26.4" x2="33.6" y2="23.6" width="0.4064" layer="1"/>
+<wire x1="24.6926" y1="19.6" x2="25.2" y2="19.6" width="0.4064" layer="1"/>
+<wire x1="25.2" y1="19.6" x2="29.2" y2="23.6" width="0.4064" layer="1"/>
+<wire x1="29.2" y1="23.6" x2="33.6" y2="23.6" width="0.4064" layer="1"/>
 </signal>
 <signal name="N$21">
@@
 <via x="34.8" y="34.8" extent="1-16" drill="1" shape="square"/>
 </signal>
+<signal name="N$38">
+<contactref element="IC1" pad="20"/>
+<contactref element="C3" pad="2"/>
+<wire x1="24.6926" y1="16.4" x2="26.8" y2="16.35" width="0.4064" layer="1"/>
+</signal>
 </signals>
